File: Power5V.sch (KiCad schematic (older format))
At the start: 5 parts

Commit message: Resolved library issues
Parts:
- C201: footprint Capacitors_SMD:C_0805 -> Capacitors_SMD:CP_Elec_6.3x5.3
Changed lines of the file:
@@
 EESchema Schematic File Version 2
+LIBS:sjaxel
+LIBS:74xgxx
+LIBS:74xx
+LIBS:ac-dc
+LIBS:actel
+LIBS:adc-dac
+LIBS:allegro
+LIBS:Altera
+LIBS:analog_devices
+LIBS:analog_switches
+LIBS:atmel
+LIBS:audio
+LIBS:battery_management
+LIBS:bbd
+LIBS:bosch
+LIBS:brooktre
+LIBS:cmos4000
+LIBS:cmos_ieee
+LIBS:conn
+LIBS:contrib
+LIBS:cypress
+LIBS:dc-dc
+LIBS:device
+LIBS:digital-audio
+LIBS:diode
+LIBS:display
+LIBS:dsp
+LIBS:elec-unifil
+LIBS:ESD_Protection
+LIBS:ftdi
+LIBS:gennum
+LIBS:graphic
+LIBS:hc11
+LIBS:intel
+LIBS:interface
+LIBS:ir
+LIBS:Lattice
+LIBS:leds
+LIBS:linear
+LIBS:logo
+LIBS:maxim
+LIBS:mechanical
+LIBS:memory
+LIBS:microchip
+LIBS:microchip_dspic33dsc
+LIBS:microchip_pic10mcu
+LIBS:microchip_pic12mcu
+LIBS:microchip_pic16mcu
+LIBS:microchip_pic18mcu
+LIBS:microchip_pic24mcu
+LIBS:microchip_pic32mcu
+LIBS:microcontrollers
+LIBS:modules
+LIBS:motor_drivers
+LIBS:motorola
+LIBS:motors
+LIBS:msp430
+LIBS:nordicsemi
+LIBS:nxp
+LIBS:nxp_armmcu
+LIBS:onsemi
+LIBS:opto
+LIBS:Oscillators
+LIBS:philips
 LIBS:power
-LIBS:device
+LIBS:powerint
+LIBS:Power_Management
+LIBS:pspice
+LIBS:references
+LIBS:regul
+LIBS:relays
+LIBS:rfcom
+LIBS:sensors
+LIBS:silabs
+LIBS:siliconi
+LIBS:stm8
+LIBS:stm32
+LIBS:supertex
+LIBS:switches
+LIBS:texas
+LIBS:transf
 LIBS:transistors
-LIBS:conn
-LIBS:linear
-LIBS:regul
-LIBS:74xx
-LIBS:cmos4000
-LIBS:adc-dac
-LIBS:memory
+LIBS:triac_thyristor
+LIBS:ttl_ieee
+LIBS:valves
+LIBS:video
+LIBS:wiznet
+LIBS:Worldsemi
+LIBS:Xicor
 LIBS:xilinx
-LIBS:microcontrollers
-LIBS:dsp
-LIBS:microchip
-LIBS:analog_switches
-LIBS:motorola
-LIBS:texas
-LIBS:intel
-LIBS:audio
-LIBS:interface
-LIBS:digital-audio
-LIBS:philips
-LIBS:display
-LIBS:cypress
-LIBS:siliconi
-LIBS:opto
-LIBS:atmel
-LIBS:contrib
-LIBS:valves
-LIBS:sjaxel
+LIBS:zetex
+LIBS:Zilog
+LIBS:driver-boostcon-cache
 EELAYER 25 0
 EELAYER END
@@
 F 0 "C201" H 3175 2750 50  0000 L CNN
 F 1 "10 uF" H 3175 2550 50  0000 L CNN
-F 2 "Capacitors_SMD:C_0805" H 3188 2500 50  0001 C CNN
+F 2 "Capacitors_SMD:CP_Elec_6.3x5.3" H 3188 2500 50  0001 C CNN
 F 3 "" H 3150 2650 50  0000 C CNN
 	1    3150 2650

Commit message: New amplifiers, fuse and general mayhem
Parts:
- C202: footprint Capacitors_SMD:C_0603 -> axel:C_0603_CustomText
- C203, C204: footprint Capacitors_SMD:C_0805 -> axel:C_0805_CustomText
Changed lines of the file:
@@
 F 0 "C203" H 5175 2850 50  0000 L CNN
 F 1 "4.7 uF" H 5175 2650 50  0000 L CNN
-F 2 "Capacitors_SMD:C_0805" H 5188 2600 50  0001 C CNN
+F 2 "axel:C_0805_CustomText" H 5188 2600 50  0001 C CNN
 F 3 "" H 5150 2750 50  0000 C CNN
 	1    5150 2750
@@
 F 0 "C204" H 5625 2850 50  0000 L CNN
 F 1 "100 nF" H 5625 2650 50  0000 L CNN
-F 2 "Capacitors_SMD:C_0805" H 5638 2600 50  0001 C CNN
+F 2 "axel:C_0805_CustomText" H 5638 2600 50  0001 C CNN
 F 3 "" H 5600 2750 50  0000 C CNN
 	1    5600 2750
@@
 F 0 "C202" H 3475 2750 50  0000 L CNN
 F 1 "100 nF" H 3475 2550 50  0000 L CNN
-F 2 "Capacitors_SMD:C_0603" H 3488 2500 50  0001 C CNN
+F 2 "axel:C_0603_CustomText" H 3488 2500 50  0001 C CNN
 F 3 "" H 3450 2650 50  0000 C CNN
 	1    3450 2650
