File: boostcon.sch (KiCad schematic (older format))
At the start: 12 parts, among them Q401 IRFH7084, Q402 BSC016N04LS

Commit message: Resolved library issues
Other:
- moved on the sheet: L401
Changed lines of the file:
@@
 EESchema Schematic File Version 2
+LIBS:sjaxel
+LIBS:74xgxx
+LIBS:74xx
+LIBS:ac-dc
+LIBS:actel
+LIBS:adc-dac
+LIBS:allegro
+LIBS:Altera
+LIBS:analog_devices
+LIBS:analog_switches
+LIBS:atmel
+LIBS:audio
+LIBS:battery_management
+LIBS:bbd
+LIBS:bosch
+LIBS:brooktre
+LIBS:cmos4000
+LIBS:cmos_ieee
+LIBS:conn
+LIBS:contrib
+LIBS:cypress
+LIBS:dc-dc
+LIBS:device
+LIBS:digital-audio
+LIBS:diode
+LIBS:display
+LIBS:dsp
+LIBS:elec-unifil
+LIBS:ESD_Protection
+LIBS:ftdi
+LIBS:gennum
+LIBS:graphic
+LIBS:hc11
+LIBS:intel
+LIBS:interface
+LIBS:ir
+LIBS:Lattice
+LIBS:leds
+LIBS:linear
+LIBS:logo
+LIBS:maxim
+LIBS:mechanical
+LIBS:memory
+LIBS:microchip
+LIBS:microchip_dspic33dsc
+LIBS:microchip_pic10mcu
+LIBS:microchip_pic12mcu
+LIBS:microchip_pic16mcu
+LIBS:microchip_pic18mcu
+LIBS:microchip_pic24mcu
+LIBS:microchip_pic32mcu
+LIBS:microcontrollers
+LIBS:modules
+LIBS:motor_drivers
+LIBS:motorola
+LIBS:motors
+LIBS:msp430
+LIBS:nordicsemi
+LIBS:nxp
+LIBS:nxp_armmcu
+LIBS:onsemi
+LIBS:opto
+LIBS:Oscillators
+LIBS:philips
 LIBS:power
-LIBS:device
+LIBS:powerint
+LIBS:Power_Management
+LIBS:pspice
+LIBS:references
+LIBS:regul
+LIBS:relays
+LIBS:rfcom
+LIBS:sensors
+LIBS:silabs
+LIBS:siliconi
+LIBS:stm8
+LIBS:stm32
+LIBS:supertex
+LIBS:switches
+LIBS:texas
+LIBS:transf
 LIBS:transistors
-LIBS:conn
-LIBS:linear
-LIBS:regul
-LIBS:74xx
-LIBS:cmos4000
-LIBS:adc-dac
-LIBS:memory
+LIBS:triac_thyristor
+LIBS:ttl_ieee
+LIBS:valves
+LIBS:video
+LIBS:wiznet
+LIBS:Worldsemi
+LIBS:Xicor
 LIBS:xilinx
-LIBS:microcontrollers
-LIBS:dsp
-LIBS:microchip
-LIBS:analog_switches
-LIBS:motorola
-LIBS:texas
-LIBS:intel
-LIBS:audio
-LIBS:interface
-LIBS:digital-audio
-LIBS:philips
-LIBS:display
-LIBS:cypress
-LIBS:siliconi
-LIBS:opto
-LIBS:atmel
-LIBS:contrib
-LIBS:valves
-LIBS:sjaxel
+LIBS:zetex
+LIBS:Zilog
+LIBS:driver-boostcon-cache
 EELAYER 25 0
 EELAYER END
@@
 U 1 1 58E528A2
 P 3750 1900
-F 0 "L401" V 3700 1900 50  0000 C CNN
-F 1 "INDUCTOR" V 3850 1900 50  0000 C CNN
+F 0 "L401" H 3750 2000 50  0000 C CNN
+F 1 "INDUCTOR" H 3750 1800 50  0000 C CNN
 F 2 "axel:SER2900" H 3750 1900 50  0001 C CNN
 F 3 "" H 3750 1900 50  0000 C CNN
 	1    3750 1900
-	0    1    1    0
+	-1   0    0    1
 $EndComp
 $Comp
@@
 Connection ~ 2300 1800
 Wire Wire Line
-	2300 1900 3450 1900
+	2300 1900 3500 1900
 Wire Wire Line
 	2300 1800 2300 2250
@@
 Connection ~ 4300 2250
 Wire Wire Line
-	4050 1900 4850 1900
+	4000 1900 4850 1900
 Wire Wire Line
 	2300 2850 2300 2550

Commit message: Syncing
Connections:
- net labels added: PowerVcc
Changed lines of the file:
@@
 Text HLabel 7400 2300 2    60   Input ~ 0
 CurrentSignal
+Text Label 2700 1900 0    60   ~ 0
+PowerVcc
 $EndSCHEMATC

Commit message: New amplifiers, fuse and general mayhem
Parts:
- removed Q401: IRFH7084, axel:PQFN_5x6_Outline-B, symbol IRFH7084
- added Q401: IRF4905S, axel:TO-263-3Lead_NoPin2, symbol IRF4905S
- added R401: 2k Ohm, axel:C_0603_CustomText, symbol R
- added R403, R404: 0.002 Ohm, axel:R-SMD-4527, symbol R
- C402, C403, C406: footprint Capacitors_SMD:C_0805 -> axel:C_0805_CustomText
- R402: renamed from R401; footprint Resistors_SMD:R_0603 -> axel:C_0603_CustomText
- renumbered R402 to R405
Connections:
- net labels added: CurrentSignal+, CurrentSignal-
- net labels removed: CurrentSignal, GroundRegulated
- wire segments 28 -> 31
Other:
- moved on the sheet: L401, R405
Changed lines of the file:
@@
 $EndDescr
-$Comp
-L IRFH7084 Q401
-U 1 1 58E5272A
-P 2100 1600
-F 0 "Q401" H 2400 1650 50  0000 R CNN
-F 1 "IRFH7084" H 2450 1350 50  0001 R CNN
-F 2 "axel:PQFN_5x6_Outline-B" H 2150 1700 50  0001 C CNN
-F 3 "" H 2100 1600 50  0000 C CNN
-	1    2100 1600
-	1    0    0    -1
-$EndComp
 $Comp
 L VCC #PWR013
 U 1 1 58E5281B
-P 1700 1400
-F 0 "#PWR013" H 1700 1250 50  0001 C CNN
-F 1 "VCC" H 1700 1550 50  0000 C CNN
-F 2 "" H 1700 1400 50  0000 C CNN
-F 3 "" H 1700 1400 50  0000 C CNN
-	1    1700 1400
-	1    0    0    -1
-$EndComp
-Text HLabel 1700 1600 0    60   Input ~ 0
+P 2300 800
+F 0 "#PWR013" H 2300 650 50  0001 C CNN
+F 1 "VCC" H 2300 950 50  0000 C CNN
+F 2 "" H 2300 800 50  0000 C CNN
+F 3 "" H 2300 800 50  0000 C CNN
+	1    2300 800
+	1    0    0    -1
+$EndComp
+Text HLabel 1700 1450 0    60   Input ~ 0
 PowerDriveSignal
 $Comp
 L INDUCTOR L401
 U 1 1 58E528A2
-P 3750 1900
-F 0 "L401" H 3750 2000 50  0000 C CNN
-F 1 "INDUCTOR" H 3750 1800 50  0000 C CNN
-F 2 "axel:SER2900" H 3750 1900 50  0001 C CNN
-F 3 "" H 3750 1900 50  0000 C CNN
-	1    3750 1900
+P 3600 1900
+F 0 "L401" H 3600 2000 50  0000 C CNN
+F 1 "INDUCTOR" H 3600 1800 50  0000 C CNN
+F 2 "axel:SER2900" H 3600 1900 50  0001 C CNN
+F 3 "" H 3600 1900 50  0000 C CNN
+	1    3600 1900
 	-1   0    0    1
 $EndComp
@@
 F 0 "C402" H 2725 2500 50  0000 L CNN
 F 1 "1 uF" H 2725 2300 50  0000 L CNN
-F 2 "Capacitors_SMD:C_0805" H 2738 2250 50  0001 C CNN
+F 2 "axel:C_0805_CustomText" H 2738 2250 50  0001 C CNN
 F 3 "" H 2700 2400 50  0000 C CNN
 	1    2700 2400
@@
 F 0 "C406" H 6325 2500 50  0000 L CNN
 F 1 "1 uF" H 6325 2300 50  0000 L CNN
-F 2 "Capacitors_SMD:C_0805" H 6338 2250 50  0001 C CNN
+F 2 "axel:C_0805_CustomText" H 6338 2250 50  0001 C CNN
 F 3 "" H 6300 2400 50  0000 C CNN
 	1    6300 2400
@@
 F 0 "C403" H 4775 2400 50  0000 L CNN
 F 1 "1 uF" H 4775 2200 50  0000 L CNN
-F 2 "Capacitors_SMD:C_0805" H 4788 2150 50  0001 C CNN
+F 2 "axel:C_0805_CustomText" H 4788 2150 50  0001 C CNN
 F 3 "" H 4750 2300 50  0000 C CNN
 	1    4750 2300
@@
 $EndComp
 $Comp
-L R R401
+L R R402
 U 1 1 58E53611
 P 4750 2650
-F 0 "R401" V 4750 2650 50  0000 C CNN
+F 0 "R402" V 4750 2650 50  0000 C CNN
 F 1 "5 Ohm" V 4850 2650 50  0000 C CNN
-F 2 "Resistors_SMD:R_0603" V 4680 2650 50  0001 C CNN
+F 2 "axel:C_0603_CustomText" V 4680 2650 50  0001 C CNN
 F 3 "" H 4750 2650 50  0000 C CNN
 	1    4750 2650
@@
 $EndComp
 $Comp
-L R R402
+L R R405
 U 1 1 58E55453
-P 7050 2500
-F 0 "R402" V 7050 2500 50  0000 C CNN
-F 1 "0.002 Ohm" V 6950 2500 50  0000 C CNN
-F 2 "axel:R-SMD-4527" V 6980 2500 50  0001 C CNN
-F 3 "" H 7050 2500 50  0000 C CNN
-	1    7050 2500
-	1    0    0    -1
-$EndComp
-$Comp
-L GNDPWR #PWR020
-U 1 1 58E555A7
-P 7050 2850
-F 0 "#PWR020" H 7050 2650 50  0001 C CNN
-F 1 "GNDPWR" H 7050 2720 50  0000 C CNN
-F 2 "" H 7050 2800 50  0000 C CNN
-F 3 "" H 7050 2800 50  0000 C CNN
-	1    7050 2850
-	1    0    0    -1
+P 7150 2100
+F 0 "R405" V 7150 2100 50  0000 C CNN
+F 1 "0.002 Ohm" V 7050 2100 50  0000 C CNN
+F 2 "axel:R-SMD-4527" V 7080 2100 50  0001 C CNN
+F 3 "" H 7150 2100 50  0000 C CNN
+	1    7150 2100
+	0    -1   -1   0
 $EndComp
 Text Label 4300 1900 0    60   ~ 0
 SwitchNode
-Text HLabel 7400 2150 2    60   Input ~ 0
-GroundRegulated
-Wire Wire Line
-	1700 1400 2350 1400
-Connection ~ 2050 1400
-Connection ~ 2150 1400
-Connection ~ 2250 1400
-Wire Wire Line
-	1700 1600 1900 1600
-Wire Wire Line
-	2200 1800 2400 1800
-Connection ~ 2300 1800
-Wire Wire Line
-	2300 1900 3500 1900
-Wire Wire Line
-	2300 1800 2300 2250
+Wire Wire Line
+	2300 1900 3350 1900
 Wire Wire Line
 	4100 2250 4400 2250
@@
 Connection ~ 4300 2250
 Wire Wire Line
-	4000 1900 4850 1900
+	3850 1900 4850 1900
 Wire Wire Line
 	2300 2850 2300 2550
@@
 Wire Wire Line
 	4750 2850 4750 2800
-Wire Wire Line
-	7050 2150 7050 2350
-Wire Wire Line
-	7050 2850 7050 2650
-Wire Wire Line
-	7050 2150 7400 2150
-Wire Wire Line
-	7400 2300 7050 2300
-Connection ~ 7050 2300
-Wire Wire Line
-	5150 1900 7400 1900
-Text HLabel 7400 1900 2    60   Input ~ 0
+Text HLabel 8200 1900 2    60   Input ~ 0
 PowerRegulated
 Connection ~ 6300 1900
@@
 $EndComp
 $Comp
-L GNDPWR #PWR021
+L GNDPWR #PWR020
 U 1 1 58F15B72
 P 5850 2850
-F 0 "#PWR021" H 5850 2650 50  0001 C CNN
+F 0 "#PWR020" H 5850 2650 50  0001 C CNN
 F 1 "GNDPWR" H 5850 2720 50  0000 C CNN
 F 2 "" H 5850 2800 50  0000 C CNN
@@
 	5850 2850 5850 2550
 Connection ~ 5850 1900
-Text HLabel 7400 2300 2    60   Input ~ 0
-CurrentSignal
+Text HLabel 6850 2100 3    60   Input ~ 0
+CurrentSignal+
 Text Label 2700 1900 0    60   ~ 0
 PowerVcc
+$Comp
+L R R404
+U 1 1 592225A6
+P 7150 1900
+F 0 "R404" V 7150 1900 50  0000 C CNN
+F 1 "0.002 Ohm" V 7050 1900 50  0000 C CNN
+F 2 "axel:R-SMD-4527" V 7080 1900 50  0001 C CNN
+F 3 "" H 7150 1900 50  0000 C CNN
+	1    7150 1900
+	0    -1   -1   0
+$EndComp
+$Comp
+L R R403
+U 1 1 59222608
+P 7150 1700
+F 0 "R403" V 7150 1700 50  0000 C CNN
+F 1 "0.002 Ohm" V 7050 1700 50  0000 C CNN
+F 2 "axel:R-SMD-4527" V 7080 1700 50  0001 C CNN
+F 3 "" H 7150 1700 50  0000 C CNN
+	1    7150 1700
+	0    -1   -1   0
+$EndComp
+Wire Wire Line
+	7300 1700 7300 2100
+Connection ~ 7300 1900
+Wire Wire Line
+	7300 1900 8200 1900
+Wire Wire Line
+	5150 1900 7000 1900
+Wire Wire Line
+	7000 1700 7000 2100
+Connection ~ 7000 1900
+Text HLabel 7450 2100 3    60   Input ~ 0
+CurrentSignal-
+Wire Wire Line
+	6850 2100 6850 1900
+Connection ~ 6850 1900
+Wire Wire Line
+	7450 2100 7450 1900
+Connection ~ 7450 1900
+$Comp
+L IRF4905S Q401
+U 1 1 592264D8
+P 2200 1500
+F 0 "Q401" H 2450 1575 50  0000 L CNN
+F 1 "IRF4905S" H 2450 1500 50  0000 L CNN
+F 2 "axel:TO-263-3Lead_NoPin2" H 2450 1425 50  0001 L CNN
+F 3 "" H 2200 1500 50  0001 L CNN
+	1    2200 1500
+	1    0    0    1
+$EndComp
+Wire Wire Line
+	1700 1450 2000 1450
+Wire Wire Line
+	2300 800  2300 1300
+Wire Wire Line
+	2300 1700 2300 2250
+$Comp
+L R R401
+U 1 1 592268B9
+P 1950 1150
+F 0 "R401" V 1950 1150 50  0000 C CNN
+F 1 "2k Ohm" V 2050 1150 50  0000 C CNN
+F 2 "axel:C_0603_CustomText" V 1880 1150 50  0001 C CNN
+F 3 "" H 1950 1150 50  0001 C CNN
+	1    1950 1150
+	1    0    0    -1
+$EndComp
+Wire Wire Line
+	1950 1450 1950 1300
+Connection ~ 1950 1450
+Wire Wire Line
+	1950 1000 1950 850
+Wire Wire Line
+	1950 850  2300 850
+Connection ~ 2300 850
 $EndSCHEMATC

Commit message: Reworked layout and added heatsink.
Parts:
- C401: value 2200 uF -> 470 uF; footprint Capacitors_ThroughHole:CP_Radial_D16.0mm_P7.50mm -> Capacitors_SMD:CP_Elec_10x10.5
- C404, C405: value 1000 uF -> 470 uF; footprint Capacitors_ThroughHole:CP_Radial_D16.0mm_P7.50mm -> Capacitors_SMD:CP_Elec_10x10.5
Other:
- moved on the sheet: L401
Changed lines of the file:
@@
 EESchema Schematic File Version 2
-LIBS:sjaxel
 LIBS:74xgxx
 LIBS:74xx
@@
 LIBS:actel
 LIBS:adc-dac
-LIBS:allegro
 LIBS:Altera
 LIBS:analog_devices
@@
 LIBS:atmel
 LIBS:audio
-LIBS:battery_management
-LIBS:bbd
-LIBS:bosch
 LIBS:brooktre
 LIBS:cmos4000
@@
 LIBS:ir
 LIBS:Lattice
-LIBS:leds
 LIBS:linear
 LIBS:logo
 LIBS:maxim
-LIBS:mechanical
 LIBS:memory
 LIBS:microchip
@@
 LIBS:microchip_pic16mcu
 LIBS:microchip_pic18mcu
-LIBS:microchip_pic24mcu
 LIBS:microchip_pic32mcu
 LIBS:microcontrollers
-LIBS:modules
 LIBS:motor_drivers
 LIBS:motorola
-LIBS:motors
 LIBS:msp430
 LIBS:nordicsemi
-LIBS:nxp
 LIBS:nxp_armmcu
 LIBS:onsemi
@@
 LIBS:transf
 LIBS:transistors
-LIBS:triac_thyristor
 LIBS:ttl_ieee
 LIBS:valves
 LIBS:video
-LIBS:wiznet
-LIBS:Worldsemi
 LIBS:Xicor
 LIBS:xilinx
-LIBS:zetex
 LIBS:Zilog
 LIBS:driver-boostcon-cache
@@
 U 1 1 58E528A2
 P 3600 1900
-F 0 "L401" H 3600 2000 50  0000 C CNN
-F 1 "INDUCTOR" H 3600 1800 50  0000 C CNN
+AR Path="/58E528A2" Ref="L401"  Part="1"
+AR Path="/58E51830/58E528A2" Ref="L401"  Part="1"
+F 0 "L401" V 3700 1900 50  0000 C CNN
+F 1 "INDUCTOR" V 3550 1900 50  0000 C CNN
 F 2 "axel:SER2900" H 3600 1900 50  0001 C CNN
 F 3 "" H 3600 1900 50  0000 C CNN
 	1    3600 1900
-	-1   0    0    1
+	0    1    1    0
 $EndComp
 $Comp
@@
 P 2300 2400
 F 0 "C401" H 2325 2500 50  0000 L CNN
-F 1 "2200 uF" H 2325 2300 50  0000 L CNN
-F 2 "Capacitors_ThroughHole:CP_Radial_D16.0mm_P7.50mm" H 2338 2250 50  0001 C CNN
+F 1 "470 uF" H 2325 2300 50  0000 L CNN
+F 2 "Capacitors_SMD:CP_Elec_10x10.5" H 2338 2250 50  0001 C CNN
 F 3 "" H 2300 2400 50  0000 C CNN
 	1    2300 2400
@@
 P 5400 2400
 F 0 "C404" H 5425 2500 50  0000 L CNN
-F 1 "1000 uF" H 5425 2300 50  0000 L CNN
-F 2 "Capacitors_ThroughHole:CP_Radial_D16.0mm_P7.50mm" H 5438 2250 50  0001 C CNN
+F 1 "470 uF" H 5425 2300 50  0000 L CNN
+F 2 "Capacitors_SMD:CP_Elec_10x10.5" H 5438 2250 50  0001 C CNN
 F 3 "" H 5400 2400 50  0000 C CNN
 	1    5400 2400
@@
 SwitchNode
 Wire Wire Line
-	2300 1900 3350 1900
-Wire Wire Line
 	4100 2250 4400 2250
 Connection ~ 4200 2250
 Connection ~ 4300 2250
-Wire Wire Line
-	3850 1900 4850 1900
 Wire Wire Line
 	2300 2850 2300 2550
@@
 P 5850 2400
 F 0 "C405" H 5875 2500 50  0000 L CNN
-F 1 "1000 uF" H 5875 2300 50  0000 L CNN
-F 2 "Capacitors_ThroughHole:CP_Radial_D16.0mm_P7.50mm" H 5888 2250 50  0001 C CNN
+F 1 "470 uF" H 5875 2300 50  0000 L CNN
+F 2 "Capacitors_SMD:CP_Elec_10x10.5" H 5888 2250 50  0001 C CNN
 F 3 "" H 5850 2400 50  0000 C CNN
 	1    5850 2400
@@
 	1950 850  2300 850
 Connection ~ 2300 850
+Wire Wire Line
+	3900 1900 4850 1900
+Wire Wire Line
+	2300 1900 3300 1900
 $EndSCHEMATC
