File: currentset.sch (KiCad schematic (older format))
At the start: 2 parts

Commit message: New amplifiers, fuse and general mayhem
Parts:
- C901: footprint Capacitors_SMD:C_0805 -> axel:C_0603_CustomText
- R901: footprint Resistors_SMD:R_0603 -> axel:C_0603_CustomText
Changed lines of the file:
@@
 F 0 "C901" H 3475 4050 50  0000 L CNN
 F 1 "100 nF" H 3475 3850 50  0000 L CNN
-F 2 "Capacitors_SMD:C_0805" H 3488 3800 50  0001 C CNN
+F 2 "axel:C_0603_CustomText" H 3488 3800 50  0001 C CNN
 F 3 "" H 3450 3950 50  0000 C CNN
 	1    3450 3950
@@
 F 0 "R901" V 2830 3600 50  0000 C CNN
 F 1 "47k" V 2750 3600 50  0000 C CNN
-F 2 "Resistors_SMD:R_0603" V 2680 3600 50  0001 C CNN
+F 2 "axel:C_0603_CustomText" V 2680 3600 50  0001 C CNN
 F 3 "" H 2750 3600 50  0000 C CNN
 	1    2750 3600
@@
 Connection ~ 3450 3600
 $Comp
-L GNDREF #PWR053
+L GNDREF #PWR050
 U 1 1 58F9242F
 P 3450 4250
-F 0 "#PWR053" H 3450 4000 50  0001 C CNN
+F 0 "#PWR050" H 3450 4000 50  0001 C CNN
 F 1 "GNDREF" H 3450 4100 50  0000 C CNN
 F 2 "" H 3450 4250 50  0000 C CNN
