File: driver.sch (KiCad schematic (older format))
At the start: 6 parts

Commit message: Resolved library issues
Connections:
- net GNDPWR: now also FDR501.1 (NC), FDR502.1 (NC)
Changed lines of the file:
@@
 EESchema Schematic File Version 2
+LIBS:sjaxel
+LIBS:74xgxx
+LIBS:74xx
+LIBS:ac-dc
+LIBS:actel
+LIBS:adc-dac
+LIBS:allegro
+LIBS:Altera
+LIBS:analog_devices
+LIBS:analog_switches
+LIBS:atmel
+LIBS:audio
+LIBS:battery_management
+LIBS:bbd
+LIBS:bosch
+LIBS:brooktre
+LIBS:cmos4000
+LIBS:cmos_ieee
+LIBS:conn
+LIBS:contrib
+LIBS:cypress
+LIBS:dc-dc
+LIBS:device
+LIBS:digital-audio
+LIBS:diode
+LIBS:display
+LIBS:dsp
+LIBS:elec-unifil
+LIBS:ESD_Protection
+LIBS:ftdi
+LIBS:gennum
+LIBS:graphic
+LIBS:hc11
+LIBS:intel
+LIBS:interface
+LIBS:ir
+LIBS:Lattice
+LIBS:leds
+LIBS:linear
+LIBS:logo
+LIBS:maxim
+LIBS:mechanical
+LIBS:memory
+LIBS:microchip
+LIBS:microchip_dspic33dsc
+LIBS:microchip_pic10mcu
+LIBS:microchip_pic12mcu
+LIBS:microchip_pic16mcu
+LIBS:microchip_pic18mcu
+LIBS:microchip_pic24mcu
+LIBS:microchip_pic32mcu
+LIBS:microcontrollers
+LIBS:modules
+LIBS:motor_drivers
+LIBS:motorola
+LIBS:motors
+LIBS:msp430
+LIBS:nordicsemi
+LIBS:nxp
+LIBS:nxp_armmcu
+LIBS:onsemi
+LIBS:opto
+LIBS:Oscillators
+LIBS:philips
 LIBS:power
-LIBS:device
+LIBS:powerint
+LIBS:Power_Management
+LIBS:pspice
+LIBS:references
+LIBS:regul
+LIBS:relays
+LIBS:rfcom
+LIBS:sensors
+LIBS:silabs
+LIBS:siliconi
+LIBS:stm8
+LIBS:stm32
+LIBS:supertex
+LIBS:switches
+LIBS:texas
+LIBS:transf
 LIBS:transistors
-LIBS:conn
-LIBS:linear
-LIBS:regul
-LIBS:74xx
-LIBS:cmos4000
-LIBS:adc-dac
-LIBS:memory
+LIBS:triac_thyristor
+LIBS:ttl_ieee
+LIBS:valves
+LIBS:video
+LIBS:wiznet
+LIBS:Worldsemi
+LIBS:Xicor
 LIBS:xilinx
-LIBS:microcontrollers
-LIBS:dsp
-LIBS:microchip
-LIBS:analog_switches
-LIBS:motorola
-LIBS:texas
-LIBS:intel
-LIBS:audio
-LIBS:interface
-LIBS:digital-audio
-LIBS:philips
-LIBS:display
-LIBS:cypress
-LIBS:siliconi
-LIBS:opto
-LIBS:atmel
-LIBS:contrib
-LIBS:valves
-LIBS:sjaxel
+LIBS:zetex
+LIBS:Zilog
+LIBS:driver-boostcon-cache
 EELAYER 25 0
 EELAYER END
@@
 	4050 2850 3950 2850
 Wire Wire Line
-	3950 2850 3950 3050
+	3950 2550 3950 3050
 Text HLabel 3300 2750 0    60   Input ~ 0
 SwitchSignal
@@
 	4000 4850 3900 4850
 Wire Wire Line
-	3900 4850 3900 5050
+	3900 4550 3900 5050
 Text HLabel 3250 4750 0    60   Input ~ 0
 PowerSignal
 Wire Wire Line
 	4000 4750 3250 4750
+Wire Wire Line
+	4050 2550 3950 2550
+Connection ~ 3950 2850
+Wire Wire Line
+	4000 4550 3900 4550
+Connection ~ 3900 4850
 $EndSCHEMATC

Commit message: New amplifiers, fuse and general mayhem
Parts:
- C501, C502: footprint Capacitors_SMD:C_0603 -> axel:C_0603_CustomText
- C503, C504: footprint Capacitors_SMD:C_0805 -> axel:C_0805_CustomText
Changed lines of the file:
@@
 $EndComp
 $Comp
-L VCC #PWR022
+L VCC #PWR021
 U 1 1 58E58F92
 P 3700 1600
-F 0 "#PWR022" H 3700 1450 50  0001 C CNN
+F 0 "#PWR021" H 3700 1450 50  0001 C CNN
 F 1 "VCC" H 3700 1750 50  0000 C CNN
 F 2 "" H 3700 1600 50  0000 C CNN
@@
 F 0 "C504" H 3425 1950 50  0000 L CNN
 F 1 "1 uF" H 3425 1750 50  0000 L CNN
-F 2 "Capacitors_SMD:C_0805" H 3438 1700 50  0001 C CNN
+F 2 "axel:C_0805_CustomText" H 3438 1700 50  0001 C CNN
 F 3 "" H 3400 1850 50  0000 C CNN
 	1    3400 1850
@@
 F 0 "C502" H 3125 1950 50  0000 L CNN
 F 1 "100 nF" H 3125 1750 50  0000 L CNN
-F 2 "Capacitors_SMD:C_0603" H 3138 1700 50  0001 C CNN
+F 2 "axel:C_0603_CustomText" H 3138 1700 50  0001 C CNN
 F 3 "" H 3100 1850 50  0000 C CNN
 	1    3100 1850
@@
 $EndComp
 $Comp
-L GNDPWR #PWR023
+L GNDPWR #PWR022
 U 1 1 58E59063
 P 3250 2250
-F 0 "#PWR023" H 3250 2050 50  0001 C CNN
+F 0 "#PWR022" H 3250 2050 50  0001 C CNN
 F 1 "GNDPWR" H 3250 2120 50  0000 C CNN
 F 2 "" H 3250 2200 50  0000 C CNN
@@
 SwitchDriveSignal
 $Comp
-L GNDPWR #PWR024
+L GNDPWR #PWR023
 U 1 1 58E59176
 P 3950 3050
-F 0 "#PWR024" H 3950 2850 50  0001 C CNN
+F 0 "#PWR023" H 3950 2850 50  0001 C CNN
 F 1 "GNDPWR" H 3950 2920 50  0000 C CNN
 F 2 "" H 3950 3000 50  0000 C CNN
@@
 $EndComp
 $Comp
-L VCC #PWR025
+L VCC #PWR024
 U 1 1 58E59460
 P 3650 3600
-F 0 "#PWR025" H 3650 3450 50  0001 C CNN
+F 0 "#PWR024" H 3650 3450 50  0001 C CNN
 F 1 "VCC" H 3650 3750 50  0000 C CNN
 F 2 "" H 3650 3600 50  0000 C CNN
@@
 F 0 "C503" H 3375 3950 50  0000 L CNN
 F 1 "1 uF" H 3375 3750 50  0000 L CNN
-F 2 "Capacitors_SMD:C_0805" H 3388 3700 50  0001 C CNN
+F 2 "axel:C_0805_CustomText" H 3388 3700 50  0001 C CNN
 F 3 "" H 3350 3850 50  0000 C CNN
 	1    3350 3850
@@
 F 0 "C501" H 3075 3950 50  0000 L CNN
 F 1 "100 nF" H 3075 3750 50  0000 L CNN
-F 2 "Capacitors_SMD:C_0603" H 3088 3700 50  0001 C CNN
+F 2 "axel:C_0603_CustomText" H 3088 3700 50  0001 C CNN
 F 3 "" H 3050 3850 50  0000 C CNN
 	1    3050 3850
@@
 $EndComp
 $Comp
-L GNDPWR #PWR026
+L GNDPWR #PWR025
 U 1 1 58E59474
 P 3200 4250
-F 0 "#PWR026" H 3200 4050 50  0001 C CNN
+F 0 "#PWR025" H 3200 4050 50  0001 C CNN
 F 1 "GNDPWR" H 3200 4120 50  0000 C CNN
 F 2 "" H 3200 4200 50  0000 C CNN
@@
 PowerDriveSignal
 $Comp
-L GNDPWR #PWR027
+L GNDPWR #PWR026
 U 1 1 58E59485
 P 3900 5050
-F 0 "#PWR027" H 3900 4850 50  0001 C CNN
+F 0 "#PWR026" H 3900 4850 50  0001 C CNN
 F 1 "GNDPWR" H 3900 4920 50  0000 C CNN
 F 2 "" H 3900 5000 50  0000 C CNN
