File: temp.sch (KiCad schematic (older format))
At the start: 2 parts

Commit message: New amplifiers, fuse and general mayhem
Parts:
- C701: footprint Capacitors_SMD:C_0603 -> axel:C_0603_CustomText
Changed lines of the file:
@@
 $EndComp
 $Comp
-L GNDD #PWR043
+L GNDD #PWR042
 U 1 1 58E7AF73
 P 5050 3300
-F 0 "#PWR043" H 5050 3050 50  0001 C CNN
+F 0 "#PWR042" H 5050 3050 50  0001 C CNN
 F 1 "GNDD" H 5050 3150 50  0000 C CNN
 F 2 "" H 5050 3300 50  0000 C CNN
@@
 	5150 2850 4900 2850
 $Comp
-L +5C #PWR044
+L +5C #PWR043
 U 1 1 58E7AFC9
 P 6650 2700
-F 0 "#PWR044" H 6650 2550 50  0001 C CNN
+F 0 "#PWR043" H 6650 2550 50  0001 C CNN
 F 1 "+5C" H 6650 2840 50  0000 C CNN
 F 2 "" H 6650 2700 50  0000 C CNN
@@
 	6050 2850 6650 2850
 $Comp
-L GNDD #PWR045
+L GNDD #PWR044
 U 1 1 58E7AFE4
 P 6200 3300
-F 0 "#PWR045" H 6200 3050 50  0001 C CNN
+F 0 "#PWR044" H 6200 3050 50  0001 C CNN
 F 1 "GNDD" H 6200 3150 50  0000 C CNN
 F 2 "" H 6200 3300 50  0000 C CNN
@@
 F 0 "C701" H 6510 3120 50  0000 L CNN
 F 1 "100 nF" H 6510 2970 50  0000 L CNN
-F 2 "Capacitors_SMD:C_0603" H 6500 3050 50  0001 C CNN
+F 2 "axel:C_0603_CustomText" H 6500 3050 50  0001 C CNN
 F 3 "" H 6500 3050 50  0000 C CNN
 	1    6500 3050
@@
 $EndComp
 $Comp
-L GNDD #PWR046
+L GNDD #PWR045
 U 1 1 58E7B064
 P 6500 3300
-F 0 "#PWR046" H 6500 3050 50  0001 C CNN
+F 0 "#PWR045" H 6500 3050 50  0001 C CNN
 F 1 "GNDD" H 6500 3150 50  0000 C CNN
 F 2 "" H 6500 3300 50  0000 C CNN
